Commit message: Adjusted imu and changed gazebo launch file to point to new ekf launch file

File: scipio_simulation/sdf/scipio_simulation_from_sdf.urdf (robot description, URDF)
Before this commit: robot scipio_simulation, 9 links, 8 joints
Links:
- removed link imu_link
- added link imu, mass 0.001
Joints:
- joint imu_joint: child imu_link -> imu; origin xyz=0 0 0 rpy=0 -0 0 -> xyz=0 0 0 rpy=3.14159 0 0

Commit message: Stereo Camera

File: scipio_simulation/sdf/scipio_simulation_from_sdf.urdf (robot description, URDF)
Before this commit: robot scipio_simulation, 9 links, 8 joints
Links:
- added link blackfly_mount_link_left, mass 1e-05; collision box size=0.05 0.05 0.05; visual box size=0.05 0.05 0.05
- added link blackfly_mount_link_right, mass 1e-05; collision box size=0.05 0.05 0.05; visual box size=0.05 0.05 0.05
- added link bumblebee_mount_link, mass 0.687646; collision mesh filename=package://lcsr_camera_models/cameras/bumblebee/bumblebee2.d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 scale=1 1 1; visual mesh filename=package://lcsr_camera_models/cameras/bumblebee/bumblebee2.d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 scale=1 1 1
- added link bumblebee_optical_link, mass 1E-6
Joints:
- added joint blackfly_mount_joint_left: type fixed, parent base_link, child blackfly_mount_link_left, origin xyz=0.05 0.35 0.8 rpy=0 0.6108652382 0.78539816339, axis -1 0 0
- added joint blackfly_mount_joint_right: type fixed, parent base_link, child blackfly_mount_link_right, origin xyz=0.05 -0.35 0.8 rpy=0 0.6108652382 -0.78539816339, axis -1 0 0
- added joint bumblebee_mount_joint: type fixed, parent base_link, child bumblebee_mount_link, origin xyz=0.2 0 0.7 rpy=1.57 3.14 -1.57, axis -1 0 0
- added joint bumblebee_optical_joint: type fixed, parent bumblebee_mount_link, child bumblebee_optical_link, origin xyz=0 0 0 rpy=3.1416 0 3.1416, axis 0 0 1
